File: kicad/pc817_bench.kicad_pcb (KiCad board)
At the start: 2 copper layers, 66 x 53.3 mm, 27 parts, among them J1 24V, e-stops, lidars, U1 PC817, U2 PC817, U3 PC817, U4 PC817

Commit message: Optional 100 nF filter capacitor on each output (C1-C4)
Between the optocoupler output and logic GND: 1 ms with the 10 k pull-up.
Board: capacitors right of the optocouplers; the two middle output tracks
move right to clear them. DRC: no errors, schematic parity OK.

Co-Authored-By: Claude Fable 5.1 <noreply@anthropic.com>
Parts:
- added C1: 100n opt., Capacitor_THT:C_Disc_D3.0mm_W1.6mm_P2.50mm, F.Cu at (147.5, 108.5)
- added C2: 100n opt., Capacitor_THT:C_Disc_D3.0mm_W1.6mm_P2.50mm, F.Cu at (147.5, 98.5)
- added C3: 100n opt., Capacitor_THT:C_Disc_D3.0mm_W1.6mm_P2.50mm, F.Cu at (147.5, 88.5)
- added C4: 100n opt., Capacitor_THT:C_Disc_D3.0mm_W1.6mm_P2.50mm, F.Cu at (147.5, 118.5)
Routing:
- net /D3: track 25.3 -> 29.9 mm
- net /D2: track 37.9 -> 41.3 mm
- net /D4: track 8.51 -> 10.9 mm
- net /D5: track 44.8 -> 47.1 mm
